File: MIDI-Guy.sch (KiCad schematic (older format))
At the start: 32 parts, among them J1 Jack-DC, J2 SJ-3523-SMT-TR, J3 SJ-3523-SMT-TR, P1 TLP291, U1 TAR5S33, U2 SAM2695, Y1 ABM8G-12.000MHZ-4Y-T3

Commit message: - Change R3 value from 470 to 220, due to receiving failure according to the transfer current spec of TLP291 - Remove panelized pcb and gerber data, since they are not maintained
Parts:
- R3: value 470? -> 220
Changed lines of the file:
@@
 EESchema Schematic File Version 4
-LIBS:SAM2695_yarou-cache
-EELAYER 29 0
+EELAYER 30 0
 EELAYER END
 $Descr A4 11693 8268
@@
 P 2950 3400
 F 0 "R3" H 2880 3354 50  0000 R CNN
-F 1 "470?" H 2880 3445 50  0000 R CNN
+F 1 "220" H 2880 3445 50  0000 R CNN
 F 2 "Resistors_SMD:R_0603_HandSoldering" V 2880 3400 50  0001 C CNN
 F 3 "~" H 2950 3400 50  0001 C CNN
@@
 	1250 6300 3400 6300
 $Comp
-L power:GNDA #PWR?
+L power:GNDA #PWR0101
 U 1 1 5CF44DA9
 P 9200 3900
-F 0 "#PWR?" H 9200 3650 50  0001 C CNN
+F 0 "#PWR0101" H 9200 3650 50  0001 C CNN
 F 1 "GNDA" H 9205 3727 50  0000 C CNN
 F 2 "" H 9200 3900 50  0001 C CNN
